Commit message: Add Final Project (Phase 1): robot_project package + sensor fusion
Phase 1 Implementation:
- New robot_project ROS 2 package for final project
- robot_localization EKF config (IMU + wheel odom fusion)
- Ground truth plugin added to URDF (p3d)
- Project launch files (project_bringup, sensor_fusion)
- Evaluation nodes (evaluation_node, map_metrics, waypoint_navigator)
- Project documentation (PROJECT_PLAN.md, README.md)

Also includes:
- HW3 corridor navigator and office world integration
- CLAUDE.md project documentation

🤖 Generated with [Claude Code](https://claude.ai/code)

Co-Authored-By: Claude <noreply@anthropic.com>

File: src/robot_hw1/urdf/p3dx_hw2.urdf.xacro (robot description, xacro)
@@ -5,37 +5,92 @@
   <xacro:property name="wheel_radius" value="0.09"/>
   <xacro:property name="wheel_width" value="0.05"/>
-  <xacro:property name="wheel_separation" value="0.33"/>
-  <xacro:property name="chassis_length" value="0.44"/>
-  <xacro:property name="chassis_width" value="0.38"/>
-  <xacro:property name="chassis_height" value="0.14"/>
-  <!-- Base Link -->
+  <xacro:property name="wheel_separation" value="0.30"/>
+  <!-- Mesh path using $(find ...) for Gazebo compatibility -->
+  <xacro:property name="mesh_path" value="$(find robot_hw1)/meshes/p3dx"/>
+  <!-- ==================== CHASSIS ==================== -->
   <link name="base_link">
     <visual>
-      <origin xyz="0 0 0.07" rpy="0 0 0"/>
-      <geometry>
-        <box size="${chassis_length} ${chassis_width} ${chassis_height}"/>
+      <origin xyz="-0.045 0 0.148" rpy="0 0 0"/>
+      <geometry>
+        <mesh filename="file://${mesh_path}/chassis.stl"/>
       </geometry>
       <material name="ChassisRed">
-        <color rgba="0.8 0.0 0.0 1.0"/>
-      </material>
-    </visual>
-    <collision>
-      <origin xyz="0 0 0.07" rpy="0 0 0"/>
-      <geometry>
-        <box size="${chassis_length} ${chassis_width} ${chassis_height}"/>
-      </geometry>
-    </collision>
-    <inertial>
-      <mass value="10.0"/>
-      <origin xyz="0 0 0.07"/>
+        <color rgba="0.851 0.0 0.0 1.0"/>
+      </material>
+    </visual>
+    <collision>
+      <origin xyz="-0.045 0 0.148" rpy="0 0 0"/>
+      <geometry>
+        <mesh filename="file://${mesh_path}/chassis.stl"/>
+      </geometry>
+    </collision>
+    <inertial>
+      <mass value="9.0"/>
+      <origin xyz="-0.045 0 0.148"/>
       <inertia ixx="0.5" ixy="0.0" ixz="0.0" iyy="0.5" iyz="0.0" izz="0.5"/>
     </inertial>
   </link>
-  <!-- Left Wheel -->
+  <!-- Top plate -->
+  <link name="top_plate">
+    <visual>
+      <origin xyz="0 0 0" rpy="0 0 0"/>
+      <geometry>
+        <mesh filename="file://${mesh_path}/top.stl"/>
+      </geometry>
+      <material name="TopBlack">
+        <color rgba="0.038 0.038 0.038 1.0"/>
+      </material>
+    </visual>
+    <collision>
+      <origin xyz="0 0 0" rpy="0 0 0"/>
+      <geometry>
+        <mesh filename="file://${mesh_path}/top.stl"/>
+      </geometry>
+    </collision>
+    <inertial>
+      <mass value="1.0"/>
+      <origin xyz="0 0 0"/>
+      <inertia ixx="0.01" ixy="0.0" ixz="0.0" iyy="0.01" iyz="0.0" izz="0.01"/>
+    </inertial>
+  </link>
+  <joint name="top_plate_joint" type="fixed">
+    <parent link="base_link"/>
+    <child link="top_plate"/>
+    <origin xyz="-0.045 0 0.234" rpy="0 0 0"/>
+  </joint>
+  <!-- Front sonar array -->
+  <link name="front_sonar">
+    <visual>
+      <origin xyz="0 0 0" rpy="0 0 0"/>
+      <geometry>
+        <mesh filename="file://${mesh_path}/front_sonar.stl"/>
+      </geometry>
+      <material name="SonarYellow">
+        <color rgba="0.8 0.8 0.0 1.0"/>
+      </material>
+    </visual>
+    <collision>
+      <origin xyz="0 0 0" rpy="0 0 0"/>
+      <geometry>
+        <mesh filename="file://${mesh_path}/front_sonar.stl"/>
+      </geometry>
+    </collision>
+    <inertial>
+      <mass value="0.1"/>
+      <origin xyz="0 0 0"/>
+      <inertia ixx="0.001" ixy="0.0" ixz="0.0" iyy="0.001" iyz="0.0" izz="0.001"/>
+    </inertial>
+  </link>
+  <joint name="front_sonar_joint" type="fixed">
+    <parent link="base_link"/>
+    <child link="front_sonar"/>
+    <origin xyz="0.109 0 0.209" rpy="0 0 0"/>
+  </joint>
+  <!-- ==================== LEFT WHEEL ==================== -->
   <link name="left_wheel">
     <visual>
-      <origin xyz="0 0 0" rpy="${M_PI/2} 0 0"/>
-      <geometry>
-        <cylinder radius="${wheel_radius}" length="${wheel_width}"/>
+      <origin xyz="0 0 0" rpy="0 0 0"/>
+      <geometry>
+        <mesh filename="file://${mesh_path}/left_wheel.stl"/>
       </geometry>
       <material name="WheelBlack">
@@ -44,7 +99,7 @@
     </visual>
     <collision>
-      <origin xyz="0 0 0" rpy="${M_PI/2} 0 0"/>
-      <geometry>
-        <cylinder radius="${wheel_radius}" length="${wheel_width}"/>
+      <origin xyz="0 0 0" rpy="0 0 0"/>
+      <geometry>
+        <mesh filename="file://${mesh_path}/left_wheel.stl"/>
       </geometry>
     </collision>
@@ -55,16 +110,37 @@
     </inertial>
   </link>
+  <link name="left_hubcap">
+    <visual>
+      <origin xyz="0 0 0" rpy="0 0 0"/>
+      <geometry>
+        <mesh filename="file://${mesh_path}/left_hubcap.stl"/>
+      </geometry>
+      <material name="HubcapYellow">
+        <color rgba="1.0 0.811 0.0 1.0"/>
+      </material>
+    </visual>
+    <inertial>
+      <mass value="0.05"/>
+      <origin xyz="0 0 0"/>
+      <inertia ixx="0.001" ixy="0.0" ixz="0.0" iyy="0.001" iyz="0.0" izz="0.001"/>
+    </inertial>
+  </link>
   <joint name="left_wheel_joint" type="continuous">
     <parent link="base_link"/>
     <child link="left_wheel"/>
-    <origin xyz="0 ${wheel_separation/2} 0" rpy="0 0 0"/>
+    <origin xyz="0 0.15 0.09" rpy="0 0 0"/>
     <axis xyz="0 1 0"/>
   </joint>
-  <!-- Right Wheel -->
+  <joint name="left_hubcap_joint" type="fixed">
+    <parent link="left_wheel"/>
+    <child link="left_hubcap"/>
+    <origin xyz="0 0 0" rpy="0 0 0"/>
+  </joint>
+  <!-- ==================== RIGHT WHEEL ==================== -->
   <link name="right_wheel">
     <visual>
-      <origin xyz="0 0 0" rpy="${M_PI/2} 0 0"/>
-      <geometry>
-        <cylinder radius="${wheel_radius}" length="${wheel_width}"/>
+      <origin xyz="0 0 0" rpy="0 0 0"/>
+      <geometry>
+        <mesh filename="file://${mesh_path}/right_wheel.stl"/>
       </geometry>
       <material name="WheelBlack">
@@ -73,7 +149,7 @@
     </visual>
     <collision>
-      <origin xyz="0 0 0" rpy="${M_PI/2} 0 0"/>
-      <geometry>
-        <cylinder radius="${wheel_radius}" length="${wheel_width}"/>
+      <origin xyz="0 0 0" rpy="0 0 0"/>
+      <geometry>
+        <mesh filename="file://${mesh_path}/right_wheel.stl"/>
       </geometry>
     </collision>
@@ -84,26 +160,74 @@
     </inertial>
   </link>
+  <link name="right_hubcap">
+    <visual>
+      <origin xyz="0 0 0" rpy="0 0 0"/>
+      <geometry>
+        <mesh filename="file://${mesh_path}/right_hubcap.stl"/>
+      </geometry>
+      <material name="HubcapYellow">
+        <color rgba="1.0 0.811 0.0 1.0"/>
+      </material>
+    </visual>
+    <inertial>
+      <mass value="0.05"/>
+      <origin xyz="0 0 0"/>
+      <inertia ixx="0.001" ixy="0.0" ixz="0.0" iyy="0.001" iyz="0.0" izz="0.001"/>
+    </inertial>
+  </link>
   <joint name="right_wheel_joint" type="continuous">
     <parent link="base_link"/>
     <child link="right_wheel"/>
-    <origin xyz="0 ${-wheel_separation/2} 0" rpy="0 0 0"/>
+    <origin xyz="0 -0.15 0.09" rpy="0 0 0"/>
     <axis xyz="0 1 0"/>
   </joint>
-  <!-- Caster Wheel -->
-  <link name="caster_wheel">
-    <visual>
+  <joint name="right_hubcap_joint" type="fixed">
+    <parent link="right_wheel"/>
+    <child link="right_hubcap"/>
+    <origin xyz="0 0 0" rpy="0 0 0"/>
+  </joint>
+  <!-- ==================== CASTER/SWIVEL WHEEL ==================== -->
+  <link name="swivel">
+    <visual>
+      <origin xyz="0 0 0" rpy="0 0 0"/>
+      <geometry>
+        <mesh filename="file://${mesh_path}/swivel.stl"/>
+      </geometry>
+      <material name="SwivelGrey">
+        <color rgba="0.5 0.5 0.5 1.0"/>
+      </material>
+    </visual>
+    <collision>
+      <origin xyz="0 0 0" rpy="0 0 0"/>
+      <geometry>
+        <mesh filename="file://${mesh_path}/swivel.stl"/>
+      </geometry>
+    </collision>
+    <inertial>
+      <mass value="0.1"/>
+      <origin xyz="0 0 0"/>
+      <inertia ixx="0.001" ixy="0.0" ixz="0.0" iyy="0.001" iyz="0.0" izz="0.001"/>
+    </inertial>
+  </link>
+  <joint name="swivel_joint" type="fixed">
+    <parent link="base_link"/>
+    <child link="swivel"/>
+    <origin xyz="-0.185 0 0.055" rpy="0 0 0"/>
+  </joint>
+  <link name="center_wheel">
+    <visual>
+      <origin xyz="0 0 0" rpy="0 0 0"/>
+      <geometry>
+        <mesh filename="file://${mesh_path}/center_wheel.stl"/>
+      </geometry>
+      <material name="CasterBlack">
+        <color rgba="0.1 0.1 0.1 1.0"/>
+      </material>
+    </visual>
+    <collision>
       <origin xyz="0 0 0" rpy="0 0 0"/>
       <geometry>
         <sphere radius="0.03"/>
       </geometry>
-      <material name="CasterGrey">
-        <color rgba="0.5 0.5 0.5 1.0"/>
-      </material>
-    </visual>
-    <collision>
-      <origin xyz="0 0 0" rpy="0 0 0"/>
-      <geometry>
-        <sphere radius="0.03"/>
-      </geometry>
     </collision>
     <inertial>
@@ -113,9 +237,31 @@
     </inertial>
   </link>
-  <joint name="caster_wheel_joint" type="fixed">
-    <parent link="base_link"/>
-    <child link="caster_wheel"/>
-    <origin xyz="-0.15 0 -0.04" rpy="0 0 0"/>
-  </joint>
+  <joint name="center_wheel_joint" type="fixed">
+    <parent link="swivel"/>
+    <child link="center_wheel"/>
+    <origin xyz="-0.026 0 -0.016" rpy="0 0 0"/>
+  </joint>
+  <link name="center_hubcap">
+    <visual>
+      <origin xyz="0 0 0" rpy="0 0 0"/>
+      <geometry>
+        <mesh filename="file://${mesh_path}/center_hubcap.stl"/>
+      </geometry>
+      <material name="HubcapYellow">
+        <color rgba="1.0 0.811 0.0 1.0"/>
+      </material>
+    </visual>
+    <inertial>
+      <mass value="0.01"/>
+      <origin xyz="0 0 0"/>
+      <inertia ixx="0.0001" ixy="0.0" ixz="0.0" iyy="0.0001" iyz="0.0" izz="0.0001"/>
+    </inertial>
+  </link>
+  <joint name="center_hubcap_joint" type="fixed">
+    <parent link="center_wheel"/>
+    <child link="center_hubcap"/>
+    <origin xyz="0 0 0" rpy="0 0 0"/>
+  </joint>
+  <!-- ==================== SENSORS ==================== -->
   <!-- RGBD Camera Link -->
   <link name="camera_link">
@@ -144,5 +290,5 @@
     <parent link="base_link"/>
     <child link="camera_link"/>
-    <origin xyz="0.15 0 0.20" rpy="0 0 0"/>
+    <origin xyz="0.15 0 0.30" rpy="0 0 0"/>
   </joint>
   <!-- Camera Optical Frame (needed for correct image orientation) -->
@@ -173,9 +319,15 @@
     <parent link="base_link"/>
     <child link="imu_link"/>
-    <origin xyz="0 0 0.10" rpy="0 0 0"/>
-  </joint>
-  <!-- Gazebo colors -->
+    <origin xyz="0 0 0.20" rpy="0 0 0"/>
+  </joint>
+  <!-- ==================== GAZEBO MATERIALS ==================== -->
   <gazebo reference="base_link">
     <material>Gazebo/Red</material>
+  </gazebo>
+  <gazebo reference="top_plate">
+    <material>Gazebo/Black</material>
+  </gazebo>
+  <gazebo reference="front_sonar">
+    <material>Gazebo/Yellow</material>
   </gazebo>
   <gazebo reference="left_wheel">
@@ -184,4 +336,7 @@
     <mu2>1.0</mu2>
   </gazebo>
+  <gazebo reference="left_hubcap">
+    <material>Gazebo/Yellow</material>
+  </gazebo>
   <gazebo reference="right_wheel">
     <material>Gazebo/Black</material>
@@ -189,8 +344,17 @@
     <mu2>1.0</mu2>
   </gazebo>
-  <gazebo reference="caster_wheel">
+  <gazebo reference="right_hubcap">
+    <material>Gazebo/Yellow</material>
+  </gazebo>
+  <gazebo reference="swivel">
     <material>Gazebo/Grey</material>
+  </gazebo>
+  <gazebo reference="center_wheel">
+    <material>Gazebo/Black</material>
     <mu1>0.1</mu1>
     <mu2>0.1</mu2>
+  </gazebo>
+  <gazebo reference="center_hubcap">
+    <material>Gazebo/Yellow</material>
   </gazebo>
   <gazebo reference="camera_link">
@@ -283,3 +447,19 @@
     </plugin>
   </gazebo>
+  <!-- ==================== GROUND TRUTH (for evaluation) ==================== -->
+  <!-- Publishes perfect odometry from Gazebo for comparing with SLAM output -->
+  <gazebo>
+    <plugin name="ground_truth_odom" filename="libgazebo_ros_p3d.so">
+      <ros>
+        <namespace>/ground_truth</namespace>
+        <remapping>odom:=odom</remapping>
+      </ros>
+      <body_name>base_link</body_name>
+      <frame_name>world</frame_name>
+      <update_rate>50.0</update_rate>
+      <xyz_offset>0 0 0</xyz_offset>
+      <rpy_offset>0 0 0</rpy_offset>
+      <gaussian_noise>0</gaussian_noise>
+    </plugin>
+  </gazebo>
 </robot>
